Commit message: Working pushing setup for three shelf-like objects

File: urdf/small_shelf_door.urdf (robot description, URDF)
Before this commit: robot small_shelf_door, 5 links, 4 joints
Joints:
- joint marker_body_joint: origin xyz=0 0 0.2065 rpy=0 0 1.57 -> xyz=-0.147 0.1575 0.2065 rpy=0 0 -1.57
- joint marker_door_joint: origin xyz=0.0075 0 0 rpy=0 0 0 -> xyz=0.0075 -0.1235 0.1255 rpy=1.57 0 1.57

Commit message: Made small shelf operation workable

File: urdf/small_shelf_door.urdf (robot description, URDF)
Before this commit: robot small_shelf_door, 5 links, 4 joints
Joints:
- joint door_joint: limit lower=0.0 upper=1.57 effort=60 velocity=0.05 -> lower=0.0 upper=1.57 effort=60 velocity=1

Commit message: Further parameterization of sync motion script. Modified CascadingQP to work with augmented gradients

File: urdf/small_shelf_door.urdf (robot description, URDF)
Before this commit: robot small_shelf_door, 5 links, 4 joints
Joints:
- joint handle_joint: origin xyz=0.0075 -0.1385 0 rpy=0 0 0 -> xyz=0.0075 -0.1385 0 rpy=1.57 0 0
